File: pcb/Split Keyboard.kicad_sch (KiCad schematic)
At the start: 3 parts

Commit message: Add other half
Designed, Placed and Routed the other half of the PCB
Parts:
- H1, H15, H2: footprint Panelization:mouse-bite-5mm-slot -> Panelization:mouse-bite-3mm-slot
Changed lines of the file:
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@@
 			)
 		)
-		(property "Footprint" "Panelization:mouse-bite-5mm-slot"
+		(property "Footprint" "Panelization:mouse-bite-3mm-slot"
 			(at 148.59 34.29 0)
 			(effects
@@
 			)
 		)
-		(property "Footprint" "Panelization:mouse-bite-5mm-slot"
+		(property "Footprint" "Panelization:mouse-bite-3mm-slot"
 			(at 148.59 25.4 0)
 			(effects
@@
 			)
 		)
-		(property "Footprint" "Panelization:mouse-bite-5mm-slot"
+		(property "Footprint" "Panelization:mouse-bite-3mm-slot"
 			(at 148.59 43.18 0)
 			(effects
